File: bessel_filter.kicad_pcb (KiCad board)
At the start: 2 copper layers, 0 parts

Commit message: progress on PCB--need to add L shield to ground connections
Parts:
- added C1: C, Capacitor_SMD:C_1206_3216Metric_Pad1.33x1.80mm_HandSolder, F.Cu at (124.5, 78.3)
- added C2: C, Capacitor_SMD:C_1206_3216Metric_Pad1.33x1.80mm_HandSolder, F.Cu at (124.5, 87.3)
- added J1: Conn_Coaxial, Connector_Coaxial:SMA_Amphenol_132289_EdgeMount, F.Cu at (115.4, 75.0)
- added J2: Conn_Coaxial, Connector_Coaxial:SMA_Amphenol_132289_EdgeMount, F.Cu at (115.4, 90.0)
- added JP1: SolderJumper_2_Bridged, Jumper:SolderJumper-2_P1.3mm_Open_TrianglePad1.0x1.5mm, F.Cu at (121.3, 81.2)
- added JP2: SolderJumper_2_Bridged, Jumper:SolderJumper-2_P1.3mm_Open_TrianglePad1.0x1.5mm, F.Cu at (121.2, 85.0)
- added L1: L_Trim, HugonLib:Coil_Craft_Unicoil_10mm, F.Cu at (132.8, 83.0)
- added REF**: MountingHole_3.5mm, MountingHole:MountingHole_3.5mm, F.Cu at (127.5, 70.5)
- added REF**: MountingHole_3.5mm, MountingHole:MountingHole_3.5mm, F.Cu at (127.5, 95.5)
Routing:
- net /GND: track 0.00 -> 18.1 mm, vias 0 -> 4
- net /sig_in: track 0.00 -> 18.1 mm
- net /sig_out: track 0.00 -> 17.8 mm
- net Net-(C1-Pad2): track 0.00 -> 2.94 mm
- net Net-(C2-Pad2): track 0.00 -> 2.71 mm
- added copper zone on B.Cu, net /GND
Other:
- board outline added: 30 x 35 mm

Commit message: PCB finished
Parts:
- L1: footprint HugonLib:Coil_Craft_Unicoil_10mm -> HugonLib:Coil_Craft_Unicoil_10mm_gnd_shield
Other:
- board text added: "0"
- board text added: "0 mm"
- board text added: "0.01 mm"
- board text added: "0.02"
- board text added: "0.035 mm"
- board text added: "0.1524 mm / 0.1524 mm"
- board text added: "0.2540 mm"
- board text added: "1"
- board text added: "1.51 mm"
- board text added: "1.6000 mm"
- board text added: "2"
- board text added: "3.3"
- board text added: "30.1000 mm x 35.1000 mm"
- board text added: "3rd Order LC Filter-Trim v1.0 2022-03-13 HugonLabs"
- board text added: "4.5"
- board text added: "B.Cu"
- board text added: "B.Mask"
- board text added: "B.Paste"
- board text added: "B.Silkscreen"
- board text added: "BOARD CHARACTERISTICS"
- board text added: "Board Thickness:"
- board text added: "Board overall dimensions:"
- board text added: "Bottom Silk Screen"
- board text added: "Bottom Solder Mask"
- board text added: "Bottom Solder Paste"
- board text added: "Castellated pads:"
- board text added: "Color"
- board text added: "Copper Finish:"
- board text added: "Copper Layer Count:"
- board text added: "Dielectric"
- board text added: "Edge card connectors:"
- board text added: "Epsilon R"
- board text added: "F.Cu"
- board text added: "F.Mask"
- board text added: "F.Paste"
- board text added: "F.Silkscreen"
- board text added: "FR4"
- board text added: "Impedance Control:"
- board text added: "Layer Name"
- board text added: "Loss Tangent"
- board text added: "Material"
- board text added: "Min hole diameter:"
- board text added: "Min track/spacing:"
- board text added: "No"
- board text added: "None"
- board text added: "Not specified"
- board text added: "Plated Board Edge:"
- board text added: "Thickness (mm)"
- board text added: "Top Silk Screen"
- board text added: "Top Solder Mask"
- board text added: "Top Solder Paste"
- board text added: "Type"
- board text added: "copper"
- board text added: "core"
